File: board/TOFE-LowSpeedIO.sch (KiCad schematic (older format))
At the start: 40 parts, among them P1 CONN_6X2, P2 CONN_6X2, P3 CONN_6X2, P4 CONN_6X2, P5 CONN_2, P6 CONN_6, SW1 SW_PUSH, SW2 SW_PUSH, SW3 SW_PUSH, SW4 SW_PUSH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

Commit message: Trying to fix the Pmod connector labeling.
Parts:
- removed P1, P2, P3, P4: CONN_6X2, ~, symbol CONN_6X2
- added P1, P2, P3, P4: PMOD-CONN_6X2, symbol PMOD-CONN_6X2
- C1, C10, C2, C3, C4: symbol C -> C-RESCUE-TOFE-LowSpeedIO
- C8, C9: symbol CP1 -> CP1-RESCUE-TOFE-LowSpeedIO
- D1, D2, D3, D5, D6, D7: symbol LED -> LED-RESCUE-TOFE-LowSpeedIO
- R1, R10, R2, R3, R6, R7, R8, R9: symbol R -> R-RESCUE-TOFE-LowSpeedIO
Connections:
- net D0: now also P4.7 (P7)
- net D1: now also P4.1 (P1)
- net D10: now also P3.8 (P8)
- net D11: now also P3.2 (P2)
- net D12: now also P3.9 (P9)
- net D13: now also P3.3 (P3)
- net D14: now also P3.10 (P10)
- net D15: now also P3.4 (P4)
- net D2: now also P4.8 (P8)
- net D3: now also P4.2 (P2)
- net D4: now also P4.9 (P9)
- net D5: now also P4.3 (P3)
- net D6: now also P4.10 (P10)
- net D7: now also P4.4 (P4)
- net D8: now also P3.7 (P7)
- net D9: now also P3.1 (P1)
- net GND: now also P1.11 (P11), P1.5 (P5), P2.11 (P11), P2.5 (P5), P3.11 (P11), P3.5 (P5), P4.11 (P11), P4.5 (P5)
- net GPIO0_N: now also P1.7 (P7)
- net GPIO0_P: now also P1.1 (P1)
- net GPIO1_N: now also P1.8 (P8)
- net GPIO1_P: now also P1.2 (P2)
- net GPIO2_N: now also P1.9 (P9)
- net GPIO2_P: now also P1.3 (P3)
- net GPIO3_N: now also P1.10 (P10)
- net GPIO3_P: now also P1.4 (P4)
- net GPIO4_N: now also P2.7 (P7)
- net GPIO4_P: now also P2.1 (P1)
- net GPIO5_N: now also P2.8 (P8)
- net GPIO5_P: now also P2.2 (P2)
- net GPIO6_N: now also P2.9 (P9)
- net GPIO6_P: now also P2.3 (P3)
- net GPIO7_N: now also P2.10 (P10)
- net GPIO7_P: now also P2.4 (P4)
- net VCC3V3: now also P1.12 (P12), P1.6 (P6), P2.12 (P12), P2.6 (P6), P3.12 (P12), P3.6 (P6), P4.12 (P12), P4.6 (P6)
